File: evilkeyboard.kicad_pcb (KiCad board)
At the start: 2 copper layers, 294.2 x 127.4 mm, 101 parts, among them SW1 RESET, SW2 RotaryEncoder_Switch, SW3 RESET, U1 TRRS, U2 RP2040_Pro_Micro, U3 TRRS, U4 RP2040_Pro_Micro

Commit message: basic pcb layout
Parts:
- removed SW2: RotaryEncoder_Switch, Keebio-Parts:RotaryEncoder_EC11
- removed SW3: RESET, Button_Switch_THT:SW_PUSH_1P1T_6x3.5mm_H4.3_APEM_MJTP1243
- added C1: 1uF, Capacitor_SMD:C_0201_0603Metric_Pad0.64x0.40mm_HandSolder, F.Cu at (157.1, 256.6)
- added C10: 1uF, Capacitor_SMD:C_0201_0603Metric_Pad0.64x0.40mm_HandSolder, F.Cu at (279.3, 229.4)
- added C2: 1uF, Capacitor_SMD:C_0201_0603Metric_Pad0.64x0.40mm_HandSolder, F.Cu at (157.1, 260.7)
- added C3: 1uF, Capacitor_SMD:C_0201_0603Metric_Pad0.64x0.40mm_HandSolder, F.Cu at (157.1, 265.9)
- added C4: 1uF, Capacitor_SMD:C_0201_0603Metric_Pad0.64x0.40mm_HandSolder, F.Cu at (157.1, 270.0)
- added C5: 100nF, Capacitor_SMD:C_0201_0603Metric_Pad0.64x0.40mm_HandSolder, F.Cu at (173.2, 167.1)
- added C6: 100nF, Capacitor_SMD:C_0201_0603Metric_Pad0.64x0.40mm_HandSolder, F.Cu at (176.1, 167.1)
- added C7: 1uF, Capacitor_SMD:C_0201_0603Metric_Pad0.64x0.40mm_HandSolder, F.Cu at (279.3, 224.1)
- added C8: 1uF, Capacitor_SMD:C_0201_0603Metric_Pad0.64x0.40mm_HandSolder, F.Cu at (279.3, 225.9)
- added C9: 1uF, Capacitor_SMD:C_0201_0603Metric_Pad0.64x0.40mm_HandSolder, F.Cu at (279.3, 227.6)
- added D100: Diode, Keebio-Parts:Diode, B.Cu at (271.2, 107.2)
- added D101: Diode, Keebio-Parts:Diode, B.Cu at (271.2, 124.8)
- added D102: Diode, Keebio-Parts:Diode, B.Cu at (289.8, 107.2)
- added D103: Diode, Keebio-Parts:Diode, B.Cu at (289.8, 124.8)
- added D104: Diode, Keebio-Parts:Diode, B.Cu at (289.8, 142.3)
- added D105: LED_WS2812B, ScottoKeebs_Components:LED_WS2812B, F.Cu at (296.1, 206.7)
- added D106: LED_WS2812B, ScottoKeebs_Components:LED_WS2812B, F.Cu at (296.1, 213.3)
- added D107: SK6812MINI, LED_SMD:LED_SK6812MINI_PLCC4_3.5x3.5mm_P1.75mm, F.Cu at (224.7, 226.9)
- added D108: SK6812MINI, LED_SMD:LED_SK6812MINI_PLCC4_3.5x3.5mm_P1.75mm, F.Cu at (224.7, 231.9)
- added D109: SK6812MINI, LED_SMD:LED_SK6812MINI_PLCC4_3.5x3.5mm_P1.75mm, F.Cu at (224.7, 237.0)
- added D110: SK6812MINI, LED_SMD:LED_SK6812MINI_PLCC4_3.5x3.5mm_P1.75mm, F.Cu at (224.7, 242.0)
- added D111: SK6812MINI, LED_SMD:LED_SK6812MINI_PLCC4_3.5x3.5mm_P1.75mm, F.Cu at (224.7, 247.1)
- added D112: Diode, Keebio-Parts:Diode, B.Cu at (308.4, 107.2)
- added D113: Diode, Keebio-Parts:Diode, B.Cu at (308.4, 142.3)
- added D114: Diode, Keebio-Parts:Diode, B.Cu at (308.4, 124.8)
- added D115: LED_WS2812B, ScottoKeebs_Components:LED_WS2812B, F.Cu at (296.1, 219.9)
- added D116: LED_WS2812B, ScottoKeebs_Components:LED_WS2812B, F.Cu at (304.6, 180.2)
- added D117: SK6812MINI, LED_SMD:LED_SK6812MINI_PLCC4_3.5x3.5mm_P1.75mm, F.Cu at (224.7, 252.1)
- added D118: SK6812MINI, LED_SMD:LED_SK6812MINI_PLCC4_3.5x3.5mm_P1.75mm, F.Cu at (224.7, 257.2)
- added D119: SK6812MINI, LED_SMD:LED_SK6812MINI_PLCC4_3.5x3.5mm_P1.75mm, F.Cu at (235.8, 225.1)
- added D120: SK6812MINI, LED_SMD:LED_SK6812MINI_PLCC4_3.5x3.5mm_P1.75mm, F.Cu at (235.8, 230.1)
- added D121: SK6812MINI, LED_SMD:LED_SK6812MINI_PLCC4_3.5x3.5mm_P1.75mm, F.Cu at (235.8, 235.2)
- added D122: LED_WS2812B, ScottoKeebs_Components:LED_WS2812B, F.Cu at (304.6, 186.8)
- added D123: LED_WS2812B, ScottoKeebs_Components:LED_WS2812B, F.Cu at (304.6, 193.5)
- added D124: SK6812MINI, LED_SMD:LED_SK6812MINI_PLCC4_3.5x3.5mm_P1.75mm, F.Cu at (235.8, 240.2)
- added D125: SK6812MINI, LED_SMD:LED_SK6812MINI_PLCC4_3.5x3.5mm_P1.75mm, F.Cu at (235.8, 245.2)
- added D126: SK6812MINI, LED_SMD:LED_SK6812MINI_PLCC4_3.5x3.5mm_P1.75mm, F.Cu at (235.8, 250.3)
- added D127: SK6812MINI, LED_SMD:LED_SK6812MINI_PLCC4_3.5x3.5mm_P1.75mm, F.Cu at (235.8, 255.3)
- added D48: Diode, Keebio-Parts:Diode, B.Cu at (136.7, 125.1)
- added D49: SK6812MINI, LED_SMD:LED_SK6812MINI_PLCC4_3.5x3.5mm_P1.75mm, F.Cu at (107.7, 95.2)
- added D50: SK6812MINI, LED_SMD:LED_SK6812MINI_PLCC4_3.5x3.5mm_P1.75mm, F.Cu at (108.4, 77.7)
- added D51: SK6812MINI, LED_SMD:LED_SK6812MINI_PLCC4_3.5x3.5mm_P1.75mm, F.Cu at (108.2, 60.2)
- added D52: SK6812MINI, LED_SMD:LED_SK6812MINI_PLCC4_3.5x3.5mm_P1.75mm, F.Cu at (89.2, 71.5)
- added D53: SK6812MINI, LED_SMD:LED_SK6812MINI_PLCC4_3.5x3.5mm_P1.75mm, F.Cu at (89.7, 89.0)
- added D54: LED_WS2812B, ScottoKeebs_Components:LED_WS2812B, F.Cu at (156.9, 227.3)
- added D55: LED_WS2812B, ScottoKeebs_Components:LED_WS2812B, F.Cu at (156.9, 233.9)
- added D56: SK6812MINI, LED_SMD:LED_SK6812MINI_PLCC4_3.5x3.5mm_P1.75mm, F.Cu at (89.7, 107.1)
- added D57: SK6812MINI, LED_SMD:LED_SK6812MINI_PLCC4_3.5x3.5mm_P1.75mm, F.Cu at (89.2, 124.1)
- added D58: SK6812MINI, LED_SMD:LED_SK6812MINI_PLCC4_3.5x3.5mm_P1.75mm, F.Cu at (70.8, 141.6)
- added D59: SK6812MINI, LED_SMD:LED_SK6812MINI_PLCC4_3.5x3.5mm_P1.75mm, F.Cu at (71.3, 124.6)
- added D60: SK6812MINI, LED_SMD:LED_SK6812MINI_PLCC4_3.5x3.5mm_P1.75mm, F.Cu at (71.3, 106.6)
- added D61: LED_WS2812B, ScottoKeebs_Components:LED_WS2812B, F.Cu at (156.9, 240.5)
- added D62: LED_WS2812B, ScottoKeebs_Components:LED_WS2812B, F.Cu at (156.9, 247.1)
- added D63: SK6812MINI, LED_SMD:LED_SK6812MINI_PLCC4_3.5x3.5mm_P1.75mm, F.Cu at (71.3, 89.6)
- added D64: SK6812MINI, LED_SMD:LED_SK6812MINI_PLCC4_3.5x3.5mm_P1.75mm, F.Cu at (52.3, 106.6)
- added D65: SK6812MINI, LED_SMD:LED_SK6812MINI_PLCC4_3.5x3.5mm_P1.75mm, F.Cu at (52.3, 124.1)
- added D66: SK6812MINI, LED_SMD:LED_SK6812MINI_PLCC4_3.5x3.5mm_P1.75mm, F.Cu at (52.3, 141.6)
- added D67: Diode, Keebio-Parts:Diode, B.Cu at (203.4, 170.2)
- added D68: LED_WS2812B, ScottoKeebs_Components:LED_WS2812B, F.Cu at (286.2, 180.0)
- added D69: LED_WS2812B, ScottoKeebs_Components:LED_WS2812B, F.Cu at (286.2, 186.6)
- added D70: SK6812MINI, LED_SMD:LED_SK6812MINI_PLCC4_3.5x3.5mm_P1.75mm, F.Cu at (217.7, 209.4)
- added D71: SK6812MINI, LED_SMD:LED_SK6812MINI_PLCC4_3.5x3.5mm_P1.75mm, F.Cu at (217.7, 216.8)
- added D72: SK6812MINI, LED_SMD:LED_SK6812MINI_PLCC4_3.5x3.5mm_P1.75mm, F.Cu at (217.7, 221.8)
- added D73: Diode, Keebio-Parts:Diode, B.Cu at (203.4, 176.3)
- added D74: Diode, Keebio-Parts:Diode, B.Cu at (215.5, 89.7)
- added D75: Diode, Keebio-Parts:Diode, B.Cu at (215.5, 107.2)
- added D76: Diode, Keebio-Parts:Diode, B.Cu at (215.5, 124.8)
- added D77: Diode, Keebio-Parts:Diode, B.Cu at (203.4, 146.4)
- added D78: LED_WS2812B, ScottoKeebs_Components:LED_WS2812B, F.Cu at (296.1, 180.2)
- added D79: LED_WS2812B, ScottoKeebs_Components:LED_WS2812B, F.Cu at (296.1, 186.8)
- added D80: Diode, Keebio-Parts:Diode, B.Cu at (234.1, 89.7)
- added D81: Diode, Keebio-Parts:Diode, B.Cu at (234.1, 107.2)
- added D82: Diode, Keebio-Parts:Diode, B.Cu at (234.1, 124.8)
- added D83: Diode, Keebio-Parts:Diode, B.Cu at (223.1, 143.2)
- added D84: SK6812MINI, LED_SMD:LED_SK6812MINI_PLCC4_3.5x3.5mm_P1.75mm, F.Cu at (217.7, 226.9)
- added D85: SK6812MINI, LED_SMD:LED_SK6812MINI_PLCC4_3.5x3.5mm_P1.75mm, F.Cu at (217.7, 231.9)
- added D86: SK6812MINI, LED_SMD:LED_SK6812MINI_PLCC4_3.5x3.5mm_P1.75mm, F.Cu at (217.7, 237.0)
- added D87: SK6812MINI, LED_SMD:LED_SK6812MINI_PLCC4_3.5x3.5mm_P1.75mm, F.Cu at (217.7, 242.0)
- added D88: Diode, Keebio-Parts:Diode, B.Cu at (252.7, 78.4)
- added D89: Diode, Keebio-Parts:Diode, B.Cu at (252.7, 95.9)
- added D90: Diode, Keebio-Parts:Diode, B.Cu at (252.7, 113.4)
- added D91: Diode, Keebio-Parts:Diode, B.Cu at (242.8, 143.3)
- added D92: LED_WS2812B, ScottoKeebs_Components:LED_WS2812B, F.Cu at (296.1, 193.5)
- added D93: LED_WS2812B, ScottoKeebs_Components:LED_WS2812B, F.Cu at (296.1, 200.1)
- added D94: SK6812MINI, LED_SMD:LED_SK6812MINI_PLCC4_3.5x3.5mm_P1.75mm, F.Cu at (217.7, 247.1)
- added D95: SK6812MINI, LED_SMD:LED_SK6812MINI_PLCC4_3.5x3.5mm_P1.75mm, F.Cu at (217.7, 252.1)
- added D96: SK6812MINI, LED_SMD:LED_SK6812MINI_PLCC4_3.5x3.5mm_P1.75mm, F.Cu at (217.7, 257.2)
- added D97: SK6812MINI, LED_SMD:LED_SK6812MINI_PLCC4_3.5x3.5mm_P1.75mm, F.Cu at (224.7, 216.8)
- added D98: SK6812MINI, LED_SMD:LED_SK6812MINI_PLCC4_3.5x3.5mm_P1.75mm, F.Cu at (224.7, 221.8)
- added D99: Diode, Keebio-Parts:Diode, B.Cu at (271.2, 89.7)
- added H1: MountingHole, MountingHole:MountingHole_2.7mm, F.Cu at (40.7, 23.7)
- added H2: MountingHole, MountingHole:MountingHole_2.7mm, F.Cu at (40.7, 32.1)
- added H3: MountingHole, MountingHole:MountingHole_2.7mm, F.Cu at (47.6, 23.7)
- added H4: MountingHole, MountingHole:MountingHole_2.7mm, F.Cu at (47.6, 32.1)
- added H5: MountingHole, MountingHole:MountingHole_2.7mm, F.Cu at (216.6, 21.4)
- added H6: MountingHole, MountingHole:MountingHole_2.7mm, F.Cu at (216.6, 29.9)
- added H7: MountingHole, MountingHole:MountingHole_2.7mm, F.Cu at (223.5, 21.4)
- added H8: MountingHole, MountingHole:MountingHole_2.7mm, F.Cu at (223.5, 29.9)
- added J1: OLED_128x32, ScottoKeebs_Components:OLED_128x32, F.Cu at (161.9, 106.2)
- added J2: OLED_128x32, ScottoKeebs_Components:OLED_128x32, F.Cu at (196.9, 123.3)
- D1: moved to F.Cu
- D15, D16, D2, D3, D31, D32, D43, D44: value Diode -> LED_WS2812B; footprint Keebio-Parts:Diode -> ScottoKeebs_Components:LED_WS2812B; moved to F.Cu
- D17, D18, D19, D20, D33, D34, D35, D36, D37, D7, D8, D9: value Diode -> SK6812MINI; footprint Keebio-Parts:Diode -> LED_SMD:LED_SK6812MINI_PLCC4_3.5x3.5mm_P1.75mm; moved to F.Cu
- S1, S10, S11, S12, S13, S14, S15, S16, S17, S18, S19, S2, S20, S21, S22, S23, S24, S25, S26, S27, S28, S29, S3, S30, S31, S32, S33, S34, S35, S36, S37, S38, S39, S4, S40, S41, S42, S43, S44, S45, S46, S47, S5, S6, S7, S8, S9: footprint ScottoKeebs_MX:MX_PCB -> keyswitches:Kailh_socket_PG1350
- SW1: value RESET -> RotaryEncoder_Switch; footprint Button_Switch_THT:SW_PUSH_1P1T_6x3.5mm_H4.3_APEM_MJTP1243 -> Keebio-Parts:RotaryEncoder_EC11
- U2, U4: value RP2040_Pro_Micro -> ~; footprint ScottoKeebs_MCU:RP2040_Pro_Micro -> Keebio-Parts:Elite-C
- moved D43 156.4 mm to (156.7, 212.3), turned to 0 degrees
- moved D47 153.5 mm to (136.7, 107.2)
- moved D46 153.3 mm to (136.7, 90.0)
- moved D45 153.2 mm to (136.7, 72.5)
- moved D44 149.1 mm to (156.9, 220.6), turned to 0 degrees
- moved D31 139.6 mm to (156.7, 199.0), turned to 0 degrees
- moved D1 139.1 mm to (135.8, 182.3), turned to 0 degrees
- moved D42 134.8 mm to (148.8, 144.1)
- moved D39 134.4 mm to (118.1, 90.0)
- moved D40 134.2 mm to (118.1, 107.6)
- moved D41 134.0 mm to (118.1, 125.1)
- moved D36 131.3 mm to (117.1, 144.2), turned to 0 degrees
- moved D38 130.4 mm to (118.1, 72.5)
- moved D32 128.3 mm to (156.7, 205.6), turned to 0 degrees
- moved D35 126.3 mm to (137.2, 142.7), turned to 0 degrees
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Connections:
- D1 pad 1: ROW2 -> Net-(D1-K)
- D1 pad 2: Net-(D1-A) -> +3.3V
- D10 pad 1: ROW3 -> Net-(D10-K)
- D10 pad 2: Net-(D10-A) -> +3.3V
- D11 pad 1: ROW4 -> ROW1
- D12 pad 1: ROW1 -> ROW2
- D13 pad 1: ROW2 -> ROW3
- D14 pad 1: ROW3 -> ROW4
- D15 pad 1: ROW4 -> Net-(D15-VDD)
- D15 pad 2: Net-(D15-A) -> Net-(D15-DOUT)
- D16 pad 1: ROW5 -> Net-(D15-VDD)
- D16 pad 2: Net-(D16-A) -> GND1
- D17 pad 1: ROW1 -> Net-(D17-DOUT)
- D17 pad 2: Net-(D17-A) -> Net-(D1-K)
- D18 pad 1: ROW2 -> Net-(D18-DOUT)
- D18 pad 2: Net-(D18-A) -> Net-(D1-K)
- D19 pad 1: ROW3 -> Net-(D19-DOUT)
- D19 pad 2: Net-(D19-A) -> Net-(D1-K)
- D2 pad 1: ROW3 -> GND1
- D2 pad 2: Net-(D2-A) -> Net-(D2-DOUT)
- D20 pad 1: ROW4 -> GND1
- D20 pad 2: Net-(D20-A) -> Net-(D1-K)
- D21 pad 1: ROW5 -> ROW1
- D22 pad 1: ROW1 -> ROW2
- D23 pad 1: ROW2 -> ROW3
- D24 pad 1: ROW3 -> ROW4
- D25 pad 1: ROW4 -> ROW5
- D26 pad 1: ROW5 -> ROW1
- D27 pad 1: ROW6 -> ROW2
- D28 pad 1: ROW7 -> ROW3
- D29 pad 1: ROW8 -> ROW4
- D3 pad 1: ROW4 -> GND1
- D3 pad 2: Net-(D3-A) -> Net-(D15-DIN)
- D30 pad 1: ROW9 -> ROW5
- D31 pad 1: ROW6 -> Net-(D31-VDD)
- D31 pad 2: Net-(D31-A) -> Net-(D31-DOUT)
- D32 pad 1: ROW7 -> Net-(D31-VDD)
- D32 pad 2: Net-(D32-A) -> GND1
- D33 pad 1: ROW8 -> Net-(D33-DOUT)
- D33 pad 2: Net-(D33-A) -> Net-(D1-K)
- D34 pad 1: ROW9 -> Net-(D34-DOUT)
- D34 pad 2: Net-(D34-A) -> Net-(D1-K)
- D35 pad 1: ROW6 -> Net-(D35-DOUT)
- D35 pad 2: Net-(D35-A) -> Net-(D1-K)
- D36 pad 1: ROW7 -> Net-(D36-DOUT)
- D36 pad 2: Net-(D36-A) -> Net-(D1-K)
- D37 pad 1: ROW8 -> Net-(D37-DOUT)
- D37 pad 2: Net-(D37-A) -> Net-(D1-K)
- D38 pad 1: ROW9 -> ROW1
- D39 pad 1: ROW6 -> ROW2
- D4 pad 1: ROW1 -> ROW2
- D40 pad 1: ROW7 -> ROW3
- D41 pad 1: ROW8 -> ROW4
- D42 pad 1: ROW6 -> ROW5
- D43 pad 1: ROW7 -> Net-(D43-VDD)
- D43 pad 2: Net-(D43-A) -> Net-(D43-DOUT)
- D44 pad 1: ROW8 -> Net-(D43-VDD)
- D44 pad 2: Net-(D44-A) -> GND1
- D45 pad 1: ROW6 -> ROW1
- D46 pad 1: ROW7 -> ROW2
- D47 pad 1: ROW8 -> ROW3
- D5 pad 1: ROW2 -> ROW3
- D6 pad 1: ROW3 -> ROW4
- D7 pad 1: ROW4 -> Net-(D7-DOUT)
- D7 pad 2: Net-(D7-A) -> Net-(D1-K)
- D8 pad 1: ROW1 -> Net-(D8-DOUT)
- D8 pad 2: Net-(D8-A) -> Net-(D1-K)
- D9 pad 1: ROW2 -> Net-(D17-DIN)
- D9 pad 2: Net-(D9-A) -> Net-(D1-K)
- S1 pad 2: Net-(D1-A) -> Net-(D4-A)
- S10 pad 2: Net-(D10-A) -> Net-(D23-A)
- S11 pad 2: Net-(D11-A) -> Net-(D24-A)
- S12 pad 1: COL4 -> COL3
- S12 pad 2: Net-(D12-A) -> Net-(D25-A)
- S13 pad 2: Net-(D13-A) -> Net-(D26-A)
- S14 pad 2: Net-(D14-A) -> Net-(D27-A)
- S15 pad 2: Net-(D15-A) -> Net-(D28-A)
- S16 pad 2: Net-(D16-A) -> Net-(D29-A)
- S17 pad 1: COL5 -> COL4
- S17 pad 2: Net-(D17-A) -> Net-(D30-A)
- S18 pad 2: Net-(D18-A) -> Net-(D38-A)
- S19 pad 2: Net-(D19-A) -> Net-(D39-A)
- S2 pad 2: Net-(D2-A) -> Net-(D5-A)
- S20 pad 2: Net-(D20-A) -> Net-(D40-A)
- S21 pad 2: Net-(D21-A) -> Net-(D41-A)
- S22 pad 1: COL6 -> COL5
- S22 pad 2: Net-(D22-A) -> Net-(D42-A)
- S23 pad 2: Net-(D23-A) -> Net-(D45-A)
- S24 pad 2: Net-(D24-A) -> Net-(D46-A)
- S25 pad 2: Net-(D25-A) -> Net-(D47-A)
- S26 pad 2: Net-(D26-A) -> Net-(D48-A)
- S27 pad 2: Net-(D27-A) -> Net-(D74-A)
- S28 pad 2: Net-(D28-A) -> Net-(D75-A)
- S29 pad 2: Net-(D29-A) -> Net-(D76-A)
- S3 pad 2: Net-(D3-A) -> Net-(D6-A)
- S30 pad 2: Net-(D30-A) -> Net-(D77-A)
- S31 pad 2: Net-(D31-A) -> Net-(D80-A)
- S32 pad 2: Net-(D32-A) -> Net-(D81-A)
- S33 pad 2: Net-(D33-A) -> Net-(D82-A)
- S34 pad 2: Net-(D34-A) -> Net-(D83-A)
- S35 pad 2: Net-(D35-A) -> Net-(D88-A)
- S36 pad 2: Net-(D36-A) -> Net-(D89-A)
- S37 pad 2: Net-(D37-A) -> Net-(D90-A)
- S38 pad 2: Net-(D38-A) -> Net-(D91-A)
- S39 pad 2: Net-(D39-A) -> Net-(D99-A)
- S4 pad 2: Net-(D4-A) -> Net-(D11-A)
- S40 pad 2: Net-(D40-A) -> Net-(D100-A)
- S41 pad 2: Net-(D41-A) -> Net-(D101-A)
- S42 pad 2: Net-(D42-A) -> Net-(D102-A)
- S43 pad 2: Net-(D43-A) -> Net-(D103-A)
- S44 pad 2: Net-(D44-A) -> Net-(D104-A)
- S45 pad 2: Net-(D45-A) -> Net-(D112-A)
- S46 pad 2: Net-(D46-A) -> Net-(D113-A)
- S47 pad 2: Net-(D47-A) -> Net-(D114-A)
- S5 pad 2: Net-(D5-A) -> Net-(D12-A)
- S6 pad 2: Net-(D6-A) -> Net-(D13-A)
- S7 pad 2: Net-(D7-A) -> Net-(D14-A)
- S8 pad 2: Net-(D8-A) -> Net-(D21-A)
- S9 pad 2: Net-(D9-A) -> Net-(D22-A)
- U1 pad 1: GND1 -> GND3
- U1 pad 2: VCC -> +3.3V
- U2 pad 1: unconnected-(U2-GP10-Pad1) -> ULED
- U2 pad 10: COL5 -> COL6
- U2 pad 11: COL6 -> ROTA
- U2 pad 12: unconnected-(U2-GP8-Pad12) -> ROTB
- U2 pad 13: unconnected-(U2-GP9-Pad13) -> ROW1
- U2 pad 14: ROTA -> ROW2
- U2 pad 15: ROTB -> ROW3
- U2 pad 16: ROTSW -> ROW4
- U2 pad 17: unconnected-(U2-GP15-Pad17) -> ROW5
- U2 pad 18: unconnected-(U2-GP16-Pad18) -> ROTSW
- U2 pad 2: unconnected-(U2-GP0-Pad2) -> BLED
- U2 pad 22: ROW5 -> unconnected-(U2-D26/A0-Pad22)
- U2 pad 23: ROW4 -> unconnected-(U2-D27/A1-Pad23)
- U2 pad 24: ROW3 -> SDA
- U2 pad 25: ROW2 -> SCL
- U2 pad 26: ROW1 -> +3.3V
- U2 pad 28: RST -> GND3
- U2 pad 29: GND1 -> unconnected-(U2-RAW-Pad29)
- U2 pad 3: unconnected-(U2-GP1-Pad3) -> GND1
- U2 pad 4: GND1 -> GND2
- U2 pad 5: GND1 -> COL1
- U2 pad 6: COL1 -> COL2
- U2 pad 7: COL2 -> COL3
- U2 pad 8: COL3 -> COL4
- U2 pad 9: COL4 -> COL5
- U3 pad 1: GND4 -> GNDR3
- U3 pad 2: VCC2 -> +3.3VR
- U4 pad 1: unconnected-(U4-GP10-Pad1) -> ULEDR
- U4 pad 10: COL11 -> COL12
- U4 pad 11: COL12 -> unconnected-(U4-D8-Pad11)
- U4 pad 14: unconnected-(U4-GP12-Pad14) -> ROW6
- U4 pad 15: unconnected-(U4-GP13-Pad15) -> ROW7
- U4 pad 16: unconnected-(U4-GP14-Pad16) -> ROW8
- U4 pad 17: unconnected-(U4-GP15-Pad17) -> ROW9
- U4 pad 2: unconnected-(U4-GP0-Pad2) -> BLEDR
- U4 pad 23: ROW9 -> unconnected-(U4-D27/A1-Pad23)
- U4 pad 24: ROW8 -> SDAR
- U4 pad 25: ROW7 -> SCLR
- U4 pad 26: ROW6 -> +3.3VR
- U4 pad 28: RST2 -> GNDR3
- U4 pad 29: GND4 -> unconnected-(U4-RAW-Pad29)
- U4 pad 3: unconnected-(U4-GP1-Pad3) -> GNDR1
- U4 pad 4: GND4 -> GNDR2
- U4 pad 5: GND4 -> COL7
- U4 pad 6: COL7 -> COL8
- U4 pad 7: COL8 -> COL9
- U4 pad 8: COL9 -> COL10
- U4 pad 9: COL10 -> COL11
Routing:
- net COL3: track 353.0 -> 0.00 mm
- net COL4: track 225.0 -> 0.00 mm
- net COL12: track 218.1 -> 0.00 mm
- net COL1: track 208.5 -> 0.00 mm
- net COL2: track 192.0 -> 0.00 mm
- net COL9: track 179.4 -> 0.00 mm
- net ROW4: track 173.6 -> 0.00 mm
- net COL5: track 168.1 -> 0.00 mm, vias 1 -> 0
- net COL11: track 166.2 -> 0.00 mm
- net COL8: track 153.7 -> 0.00 mm
- net ROW3: track 152.9 -> 0.00 mm
- net ROW8: track 145.6 -> 0.00 mm
- net ROW2: track 138.6 -> 0.00 mm
- net COL10: track 138.2 -> 0.00 mm
- net ROW7: track 136.0 -> 0.00 mm
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Other:
- board outline removed
