File: evilkeyboard.kicad_sch (KiCad schematic)
At the start: 254 parts, among them J1 OLED_128x32, J2 OLED_128x32, SW2 RotaryEncoder_Switch, U1 TRRS, U3 TRRS

Commit message: Revision 1
Parts:
- removed C10, C11, C12, C13, C14, C15, C16, C17, C18, C19, C20, C21, C22, C23, C24, C25, C26, C27, C28, C29, C30, C31, C32, C33, C34, C35, C36, C37, C38, C39, C40, C41, C42, C43, C44, C45, C46, C47, C48, C51, C52, C53, C55, C56, C57, C59, C60, C61, C63, C64, C65, C66, C67, C68, C69, C70, C71, C72, C73, C74: C100nF, symbol Device:C
- removed D61: LED_WS2812B, ScottoKeebs_Components:LED_WS2812B, symbol ScottoKeebs:LED_WS2812B
- removed R2, R3, R4, R5: R100, symbol Device:R
- added C49: 1uF, symbol Device:C
- added D101, D105, D114, D61: Diode, Keebio-Parts:Diode, symbol ScottoKeebs:Placeholder_Diode
- added D109: LED_WS2812B, ScottoKeebs_Components:LED_WS2812B, symbol ScottoKeebs:LED_WS2812B
- C1, C2: value C0.1u -> 100nF
- C3, C4, C5, C6, C7, C8, C9: value C100nF -> 1uF
Connections:
- net GNDR is gone; now on net GND: D62.3 (VSS), D63.3 (VSS), D64.3 (VSS), D65.3 (VSS), D66.3 (VSS), D67.3 (VSS), D68.3 (VSS), D69.3 (VSS), D70.3 (VSS), D71.3 (VSS), D72.3 (VSS), J1.1 (GND), U3.1 (SLEEVE), U4.28 (GND), U4.3 (D10/GND), U4.4 (D11/GND)
- net +3.3V: now also D101.2 (A), D105.2 (A); no longer C3.1, C4.1, C5.1, C6.1, C7.1, C8.1, C9.1, D100.4 (VDD), D102.4 (VDD), D103.4 (VDD), D104.4 (VDD), D106.4 (VDD), D107.4 (VDD), D108.4 (VDD), D110.4 (VDD), D111.4 (VDD), D112.4 (VDD), D113.4 (VDD), D115.4 (VDD), D116.4 (VDD), D117.4 (VDD), D118.4 (VDD), D120.4 (VDD), D121.4 (VDD), D122.4 (VDD), D123.4 (VDD), D48.1 (VDD), D49.4 (VDD), D50.1 (VDD), D51.1 (VDD), D52.1 (VDD), D53.1 (VDD), D54.1 (VDD), D55.1 (VDD), D56.1 (VDD), D57.1 (VDD), D58.1 (VDD), D59.1 (VDD), D60.1 (VDD), D73.4 (VDD), D74.4 (VDD), D75.4 (VDD), D76.4 (VDD), D77.4 (VDD), D78.4 (VDD), D79.4 (VDD), D80.4 (VDD), D81.4 (VDD), D82.4 (VDD), D83.4 (VDD), D84.4 (VDD), D85.4 (VDD), D86.4 (VDD), D87.4 (VDD), D88.4 (VDD), D89.4 (VDD), D90.4 (VDD), D91.4 (VDD), D92.4 (VDD), D93.4 (VDD), D94.4 (VDD), D95.4 (VDD), D96.4 (VDD), D97.4 (VDD), D98.4 (VDD), D99.4 (VDD)
- net +3.3VR: now also D114.2 (A), D61.2 (A); no longer D62.1 (VDD), D63.1 (VDD), D64.1 (VDD), D65.1 (VDD), D66.1 (VDD), D67.1 (VDD), D68.1 (VDD), D69.1 (VDD), D70.1 (VDD), D71.1 (VDD), D72.1 (VDD)
- net GND: now also C49.2, D109.3 (VSS)
- net ULED: now also D55.4 (DIN)
- net ULEDR: now also D62.4 (DIN)
- net at D67.4 (DIN): now also D65.2 (DOUT)
- net at D71.2 (DOUT): now also D109.4 (DIN); no longer D68.4 (DIN)
- net at D66.2 (DOUT): now also D63.4 (DIN)
- net at D69.4 (DIN): now also D72.2 (DOUT); no longer D67.2 (DOUT)
- net at D48.4 (DIN): now also D60.2 (DOUT)
- new net: C6.1, D109.1 (VDD), D61.1 (K), D62.1 (VDD), D63.1 (VDD), D64.1 (VDD), D65.1 (VDD), D66.1 (VDD), D67.1 (VDD), D68.1 (VDD), D69.1 (VDD), D70.1 (VDD), D71.1 (VDD), D72.1 (VDD)
- new net: C3.1, C4.1, C5.1, D101.1 (K), D49.4 (VDD), D73.4 (VDD), D74.4 (VDD), D75.4 (VDD), D76.4 (VDD), D77.4 (VDD), D78.4 (VDD), D79.4 (VDD), D80.4 (VDD), D81.4 (VDD), D82.4 (VDD), D83.4 (VDD), D84.4 (VDD), D85.4 (VDD), D86.4 (VDD), D87.4 (VDD), D88.4 (VDD), D89.4 (VDD), D90.4 (VDD), D91.4 (VDD), D92.4 (VDD), D93.4 (VDD), D94.4 (VDD), D95.4 (VDD), D96.4 (VDD), D97.4 (VDD)
- new net: C7.1, C8.1, C9.1, D100.4 (VDD), D102.4 (VDD), D103.4 (VDD), D104.4 (VDD), D106.4 (VDD), D107.4 (VDD), D108.4 (VDD), D110.4 (VDD), D111.4 (VDD), D112.4 (VDD), D113.4 (VDD), D114.1 (K), D115.4 (VDD), D116.4 (VDD), D117.4 (VDD), D118.4 (VDD), D120.4 (VDD), D121.4 (VDD), D122.4 (VDD), D123.4 (VDD), D98.4 (VDD), D99.4 (VDD)
- new net: C49.1, D105.1 (K), D48.1 (VDD), D50.1 (VDD), D51.1 (VDD), D52.1 (VDD), D53.1 (VDD), D54.1 (VDD), D55.1 (VDD), D56.1 (VDD), D57.1 (VDD), D58.1 (VDD), D59.1 (VDD), D60.1 (VDD)
- new net: D67.2 (DOUT), D68.4 (DIN)
- no-connect marks 18 -> 16

Commit message: basic pcb layout
Parts:
- removed C6: 1uF, symbol Device:C
- removed D100, D102, D103, D104, D106, D112, D113, D115, D116, D122, D123, D73, D74, D75, D76, D78, D79, D80, D81, D82, D88, D90, D91, D92, D93, D99: SK6812MINI, LED_SMD:LED_SK6812MINI_PLCC4_3.5x3.5mm_P1.75mm, symbol LED:SK6812MINI
- removed D109, D48, D50, D51, D52, D53, D63, D64, D65, D66, D67, D70, D71, D72: LED_WS2812B, ScottoKeebs_Components:LED_WS2812B, symbol ScottoKeebs:LED_WS2812B
- removed D114, D61: Diode, Keebio-Parts:Diode, symbol ScottoKeebs:Placeholder_Diode
- removed H1, H2, H3, H4: MountingHole, MountingHole:MountingHole_2.7mm, symbol Mechanical:MountingHole
- removed R1: R1K, symbol Device:R
- added C10: 1uF, Capacitor_SMD:C_0201_0603Metric_Pad0.64x0.40mm_HandSolder, symbol Device:C
- added D105, D106, D115, D116, D122, D123, D43, D44, D55, D61, D78, D79, D92, D93: LED_WS2812B, ScottoKeebs_Components:LED_WS2812B, symbol ScottoKeebs:LED_WS2812B
- added D109, D119, D124, D125, D126, D127, D17, D18, D19, D20, D33, D34, D35, D36, D37, D50, D51, D52, D53, D56, D57, D58, D59, D60, D63, D64, D65, D66, D70, D71, D72: SK6812MINI, LED_SMD:LED_SK6812MINI_PLCC4_3.5x3.5mm_P1.75mm, symbol LED:SK6812MINI
- added D67, D73: Diode, Keebio-Parts:Diode, symbol ScottoKeebs:Placeholder_Diode
- added H5, H6, H7, H8: MountingHole, MountingHole:MountingHole_2.7mm, symbol Mechanical:MountingHole
- C1: renamed from C49; footprint (none) -> Capacitor_SMD:C_0201_0603Metric_Pad0.64x0.40mm_HandSolder
- C2: renamed from C5; footprint (none) -> Capacitor_SMD:C_0201_0603Metric_Pad0.64x0.40mm_HandSolder
- C3: renamed from C4; footprint (none) -> Capacitor_SMD:C_0201_0603Metric_Pad0.64x0.40mm_HandSolder
- C4: renamed from C3; footprint (none) -> Capacitor_SMD:C_0201_0603Metric_Pad0.64x0.40mm_HandSolder
- C5: renamed from C2; footprint (none) -> Capacitor_SMD:C_0201_0603Metric_Pad0.64x0.40mm_HandSolder
- C6: renamed from C1; footprint (none) -> Capacitor_SMD:C_0201_0603Metric_Pad0.64x0.40mm_HandSolder
- C7, C8, C9: footprint (none) -> Capacitor_SMD:C_0201_0603Metric_Pad0.64x0.40mm_HandSolder
- S1, S10, S11, S2, S27, S28, S29, S3, S30, S31, S32, S33, S34, S35, S36, S37, S38, S39, S4, S40, S41, S42, S43, S44, S45, S46, S47, S5, S6, S7, S8, S9: footprint ScottoKeebs_MX:MX_PCB -> keyswitches:Kailh_socket_PG1350
- S12: renamed from S16; footprint ScottoKeebs_MX:MX_PCB -> keyswitches:Kailh_socket_PG1350
- S13: renamed from S12; footprint ScottoKeebs_MX:MX_PCB -> keyswitches:Kailh_socket_PG1350
- S14: renamed from S13; footprint ScottoKeebs_MX:MX_PCB -> keyswitches:Kailh_socket_PG1350
- S15: renamed from S14; footprint ScottoKeebs_MX:MX_PCB -> keyswitches:Kailh_socket_PG1350
- S16: renamed from S15; footprint ScottoKeebs_MX:MX_PCB -> keyswitches:Kailh_socket_PG1350
- S17: renamed from S21; footprint ScottoKeebs_MX:MX_PCB -> keyswitches:Kailh_socket_PG1350
- S18: renamed from S17; footprint ScottoKeebs_MX:MX_PCB -> keyswitches:Kailh_socket_PG1350
- S19: renamed from S18; footprint ScottoKeebs_MX:MX_PCB -> keyswitches:Kailh_socket_PG1350
- S20: renamed from S19; footprint ScottoKeebs_MX:MX_PCB -> keyswitches:Kailh_socket_PG1350
- S21: renamed from S20; footprint ScottoKeebs_MX:MX_PCB -> keyswitches:Kailh_socket_PG1350
- S22: renamed from S26; footprint ScottoKeebs_MX:MX_PCB -> keyswitches:Kailh_socket_PG1350
- S23: renamed from S22; footprint ScottoKeebs_MX:MX_PCB -> keyswitches:Kailh_socket_PG1350
- S24: renamed from S23; footprint ScottoKeebs_MX:MX_PCB -> keyswitches:Kailh_socket_PG1350
- S25: renamed from S24; footprint ScottoKeebs_MX:MX_PCB -> keyswitches:Kailh_socket_PG1350
- S26: renamed from S25; footprint ScottoKeebs_MX:MX_PCB -> keyswitches:Kailh_socket_PG1350
- U2, U4: footprint ScottoKeebs_MCU:RP2040_Pro_Micro -> Keebio-Parts:Elite-C
- renumbered D101 to D1, D105 to D10, D40 to D100, D41 to D101, D42 to D102, D43 to D103, D44 to D104, D4 to D11, D45 to D112, D46 to D113, D47 to D114, D5 to D12, D6 to D13, D7 to D14, D57 to D15, D58 to D16, D55 to D2, D8 to D21, D9 to D22, D10 to D23, D11 to D24, D16 to D25, D12 to D26, D13 to D27, D14 to D28, D15 to D29, D56 to D3, D21 to D30, D59 to D31, D60 to D32, D17 to D38, D18 to D39, D1 to D4, D19 to D40, D20 to D41, D26 to D42, D22 to D45, D23 to D46, D24 to D47, D25 to D48, D2 to D5, D3 to D6, D77 to D7, D27 to D74, D28 to D75, D29 to D76, D30 to D77, D83 to D8, D31 to D80, D32 to D81, D33 to D82, D34 to D83, D35 to D88, D36 to D89, D89 to D9, D37 to D90, D38 to D91, D39 to D99, H5 to H1, H6 to H2, H7 to H3, H8 to H4, J2 to J1, J1 to J2, SW2 to SW1
Connections:
- net +3.3VR: now also D67.2 (A), D73.2 (A)
- net BLED: now also D7.3 (DIN); no longer D49.3 (DIN)
- net BLEDR: now also D70.3 (DIN); no longer D98.3 (DIN)
- net ULEDR: now also D68.4 (DIN); no longer D62.4 (DIN)
- net GND3: now reaches SW1.S2
- net GND3: now also C5.2, C6.1, SW1.C, U1.1 (SLEEVE), U2.28 (GND)
- net GND1R: now reaches D68.1 (VDD), D69.1 (VDD)
- net GND1R: now also C7.2, C8.2, C9.2, D107.4 (VDD), D108.4 (VDD), D110.4 (VDD), D111.4 (VDD), D117.4 (VDD), D118.4 (VDD), D120.4 (VDD), D121.4 (VDD), D87.1 (DOUT), D94.3 (DIN), D94.4 (VDD), D95.4 (VDD), D96.4 (VDD), D97.4 (VDD), D98.4 (VDD), C10.2, D105.4 (DIN), D106.2 (DOUT), D109.4 (VDD), D115.4 (DIN), D116.2 (DOUT), D119.4 (VDD), D122.1 (VDD), D122.4 (DIN), D123.1 (VDD), D124.4 (VDD), D125.4 (VDD), D126.4 (VDD), D127.4 (VDD), D70.4 (VDD), D71.4 (VDD), D72.4 (VDD), D79.2 (DOUT), D92.4 (DIN), D93.2 (DOUT); no longer D62.1 (VDD)
- net at D97.1 (DOUT): now also D98.3 (DIN)
- net at D108.3 (DIN): now also D107.1 (DOUT)
- net at D120.1 (DOUT): now also D121.3 (DIN)
- net at D15.2 (DOUT): now also D16.4 (DIN); no longer D31.4 (DIN)
- net at D15.4 (DIN): now also D3.2 (DOUT); no longer D2.2 (DOUT)
- net at D117.3 (DIN): now also D111.1 (DOUT)
- net at D108.1 (DOUT): now also D109.3 (DIN)
- net at D9.1 (DOUT): now also D17.3 (DIN)
- net at D9.3 (DIN): now also D8.1 (DOUT)
- net at D118.1 (DOUT): now also D119.3 (DIN)
- net at D118.3 (DIN): now also D117.1 (DOUT)
- net at D7.1 (DOUT): now also D8.3 (DIN)
- net at D69.4 (DIN): now also D68.2 (DOUT)
- net at D84.3 (DIN): now also D72.1 (DOUT); no longer D8.1 (DOUT)
- net at D121.1 (DOUT): now also D124.3 (DIN)
- net GND1: now reaches D54.4 (DIN)
- net GND1: now also C1.2, C2.2, C3.2, C4.2, D16.2 (DOUT), D2.1 (VDD), D3.1 (VDD), D31.4 (DIN), D32.2 (DOUT), D49.4 (VDD), D62.1 (VDD), D7.4 (VDD), D8.4 (VDD), D9.4 (VDD), U2.3 (D10/GND), D20.1 (DOUT), D33.3 (DIN), D33.4 (VDD), D34.4 (VDD), D35.4 (VDD), D36.4 (VDD), D37.4 (VDD), D43.4 (DIN), D44.2 (DOUT), D50.4 (VDD), D51.4 (VDD), D52.4 (VDD), D53.4 (VDD), D55.2 (DOUT), D56.4 (VDD), D57.4 (VDD), D58.4 (VDD), D59.4 (VDD), D60.4 (VDD), D61.1 (VDD), D61.4 (DIN), D63.4 (VDD), D64.4 (VDD), D65.4 (VDD), D66.4 (VDD)
- net at D3.4 (DIN): now also D2.2 (DOUT); no longer D31.2 (DOUT)
- net at D32.4 (DIN): now also D31.2 (DOUT); no longer D16.2 (DOUT)
- net at D54.2 (DOUT): now also D55.4 (DIN)
- net at D111.3 (DIN): now also D110.1 (DOUT); no longer D107.1 (DOUT)
- net at D107.3 (DIN): now also D98.1 (DOUT)
- net at D120.3 (DIN): now also D119.1 (DOUT)
- net at D110.3 (DIN): now also D109.1 (DOUT)
- net at D69.2 (DOUT): now also D78.4 (DIN)
- net at D49.1 (DOUT): now also D50.3 (DIN)
- removed net GND: C1.2, C2.2, C3.2, C4.2, C5.2, C6.1, C7.2, C8.2, C9.2, D107.2 (VSS), D108.2 (VSS), D110.2 (VSS), D111.2 (VSS), D117.2 (VSS), D118.2 (VSS), D120.2 (VSS), D121.2 (VSS), D15.3 (VSS), D16.3 (VSS), D2.3 (VSS), D3.3 (VSS), D31.3 (VSS), D32.3 (VSS), D49.2 (VSS), D54.3 (VSS), D62.3 (VSS), D68.3 (VSS), D69.3 (VSS), D7.2 (VSS), D8.2 (VSS), D84.2 (VSS), D85.2 (VSS), D86.2 (VSS), D87.2 (VSS), D9.2 (VSS), D94.2 (VSS), D95.2 (VSS), D96.2 (VSS), D97.2 (VSS), D98.2 (VSS), J1.1 (GND), J2.1 (GND), SW1.C, U1.1 (SLEEVE), U2.28 (GND), U2.3 (D10/GND), U2.4 (D11/GND), U3.1 (SLEEVE), U4.28 (GND), U4.3 (D10/GND), U4.4 (D11/GND)
- new net: D59.1 (DOUT), D60.3 (DIN)
- new net: C2.1, C3.1, C4.1, D1.1 (K), D17.2 (VSS), D18.2 (VSS), D19.2 (VSS), D20.2 (VSS), D33.2 (VSS), D34.2 (VSS), D35.2 (VSS), D36.2 (VSS), D37.2 (VSS), D49.2 (VSS), D50.2 (VSS), D51.2 (VSS), D52.2 (VSS), D53.2 (VSS), D56.2 (VSS), D57.2 (VSS), D58.2 (VSS), D59.2 (VSS), D60.2 (VSS), D63.2 (VSS), D64.2 (VSS), D65.2 (VSS), D66.2 (VSS), D7.2 (VSS), D8.2 (VSS), D9.2 (VSS)
- new net: D58.1 (DOUT), D59.3 (DIN)
- new net: C10.1, C8.1, C9.1, D107.2 (VSS), D108.2 (VSS), D109.2 (VSS), D110.2 (VSS), D111.2 (VSS), D117.2 (VSS), D118.2 (VSS), D119.2 (VSS), D120.2 (VSS), D121.2 (VSS), D124.2 (VSS), D125.2 (VSS), D126.2 (VSS), D127.2 (VSS), D67.1 (K), D70.2 (VSS), D71.2 (VSS), D72.2 (VSS), D84.2 (VSS), D85.2 (VSS), D86.2 (VSS), D87.2 (VSS), D94.2 (VSS), D95.2 (VSS), D96.2 (VSS), D97.2 (VSS), D98.2 (VSS)
- new net: D84.4 (VDD), D85.4 (VDD), D86.4 (VDD), D87.4 (VDD)
- new net: D15.1 (VDD), D16.1 (VDD)
- new net: C1.1, D10.1 (K), D15.3 (VSS), D16.3 (VSS), D2.3 (VSS), D3.3 (VSS), D31.3 (VSS), D32.3 (VSS), D43.3 (VSS), D44.3 (VSS), D54.3 (VSS), D55.3 (VSS), D61.3 (VSS), D62.3 (VSS)
- new net: D35.1 (DOUT), D36.3 (DIN)
- new net: D34.1 (DOUT), D35.3 (DIN)
- new net: D19.1 (DOUT), D20.3 (DIN)
- new net: D17.4 (VDD), D18.4 (VDD), D19.4 (VDD), D20.4 (VDD)
- new net: C7.1, D105.3 (VSS), D106.3 (VSS), D115.3 (VSS), D116.3 (VSS), D122.3 (VSS), D123.3 (VSS), D68.3 (VSS), D69.3 (VSS), D73.1 (K), D78.3 (VSS), D79.3 (VSS), D92.3 (VSS), D93.3 (VSS)
- new net: D92.1 (VDD), D93.1 (VDD)
- new net: D92.2 (DOUT), D93.4 (DIN)
- new net: D78.1 (VDD), D79.1 (VDD)
- new net: D78.2 (DOUT), D79.4 (DIN)
- new net: D37.1 (DOUT), D49.3 (DIN)
- new net: D60.1 (DOUT), D63.3 (DIN)
- new net: D122.2 (DOUT), D123.4 (DIN)
- new net: D56.1 (DOUT), D57.3 (DIN)
- new net: D53.1 (DOUT), D56.3 (DIN)
- new net: D65.1 (DOUT), D66.3 (DIN)
- new net: D64.1 (DOUT), D65.3 (DIN)
- new net: D115.1 (VDD), D116.1 (VDD)
- new net: D115.2 (DOUT), D116.4 (DIN)
- new net: D36.1 (DOUT), D37.3 (DIN)
- new net: D63.1 (DOUT), D64.3 (DIN)
- new net: D124.1 (DOUT), D125.3 (DIN)
- new net: D50.1 (DOUT), D51.3 (DIN)
- new net: D17.1 (DOUT), D18.3 (DIN)
- new net: D61.2 (DOUT), D62.4 (DIN)
- new net: D43.1 (VDD), D44.1 (VDD)
- new net: D43.2 (DOUT), D44.4 (DIN)
- new net: D33.1 (DOUT), D34.3 (DIN)
- new net: D71.1 (DOUT), D72.3 (DIN)
- new net: D70.1 (DOUT), D71.3 (DIN)
- new net: D57.1 (DOUT), D58.3 (DIN)
- new net: D52.1 (DOUT), D53.3 (DIN)
- new net: D51.1 (DOUT), D52.3 (DIN)
- new net: D125.1 (DOUT), D126.3 (DIN)
- new net: D54.1 (VDD), D55.1 (VDD)
- new net: D105.1 (VDD), D106.1 (VDD)
- new net: D105.2 (DOUT), D106.4 (DIN)
- new net: D126.1 (DOUT), D127.3 (DIN)
- new net: D31.1 (VDD), D32.1 (VDD)
- new net: D18.1 (DOUT), D19.3 (DIN)
- new net GND2: J1.1 (GND), U2.4 (D11/GND)
- new net GNDR1: U4.3 (D10/GND)
- new net GNDR2: U4.4 (D11/GND)
- new net GNDR3: J2.1 (GND), U3.1 (SLEEVE), U4.28 (GND)
Other:
- moved on the sheet: C1, C2, C3, C4, C5, C6, D1, D10, D100, D101, D102, D103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
